File: hardware/101.kicad_sch (KiCad schematic)
At the start: 8 parts

Commit message: update: 原理图好了
Parts:
- removed SW? (x2): SW_Push, symbol Switch:SW_Push
- removed U?: ZJY154T-PG04, chenxuuu_Module:ZJY154T-PG04(ST7789-240x240), symbol chenxuuu_Library:ZJY154T-PG04
- removed U?: SC662, Package_TO_SOT_SMD:SOT-23, symbol chenxuuu_Library:SC662
- added AE1: Antenna_Shield, RF_Antenna:Texas_SWRA117D_2.4GHz_Left, symbol Device:Antenna_Shield
- added C1, C2: 15p, Capacitor_SMD:C_0402_1005Metric, symbol Device:C
- added C10, C11, C12, C13, C3, C7: 1uF, Capacitor_SMD:C_0402_1005Metric, symbol Device:C
- added C14, C9: 4.7uF, Capacitor_SMD:C_0402_1005Metric, symbol Device:C
- added C15: Cap_0.1uf_0402_16V_X7R, Capacitor_SMD:C_0402_1005Metric, symbol Airm2m_RCL:Cap_0.1uf_0402_16V_X7R
- added C4: 10uF, Capacitor_SMD:C_0402_1005Metric, symbol Device:C
- added C5: 100nf, Capacitor_SMD:C_0402_1005Metric, symbol Device:C
- added C6: 104, Capacitor_SMD:C_0402_1005Metric, symbol Device:C
- added C8: 102, Capacitor_SMD:C_0402_1005Metric, symbol Device:C
- added D1: LED, symbol Device:LED
- added D2: SS14, Diode_SMD:D_SMA, symbol Device:D
- added J2: Conn_01x04_Male, symbol Connector:Conn_01x04_Male
- added J3: ST7735S-0.96TFT-13P, chenxuuu_Module:ST7735S-0.96TFT-13P, symbol chenxuuu_Library:ST7735S-0.96TFT-13P
- added R1, R2: 100K, Resistor_SMD:R_0402_1005Metric, symbol Device:R
- added R10: 10R, Resistor_SMD:R_0402_1005Metric, symbol Device:R
- added R11, R12, R13, R14, R15: 100K, symbol Device:R
- added R3, R4: 5.1K, symbol Device:R
- added R5: 5.1K, Resistor_SMD:R_0402_1005Metric, symbol Device:R
- added R6: 1K, Resistor_SMD:R_0402_1005Metric, symbol Device:R
- added R7: 0.5R, Resistor_SMD:R_0402_1005Metric, symbol Device:R
- added R8: 1R, Resistor_SMD:R_0402_1005Metric, symbol Device:R
- added R9: 2K, Resistor_SMD:R_0402_1005Metric, symbol Device:R
- added SW2: SW_ON/OFF, symbol Switch:SW_Push
- added U1: 4A2D, Package_TO_SOT_SMD:SOT-23-5, symbol chenxuuu_Library:LDO_5PIN
- added U2: CH330N, Package_SO:SOIC-8_3.9x4.9mm_P1.27mm, symbol chenxuuu_Library:CH330N
- added U4: HX4064A, Package_TO_SOT_SMD:SOT-23-5, symbol chenxuuu_Library:HX4064A
- added Y1: 40M, Crystal:Crystal_SMD_3225-4Pin_3.2x2.5mm, symbol Device:Crystal_GND24
- gave numbers to parts that had none: 4
Connections:
- net KEY: now reaches SW1.1
- net KEY: now also U3.14 (PA1/JTAG_CK/I2C_SCL/PWM3/I2S_LRCK/ADC0)
- net GND: now reaches SW1.2
- net GND: now also J1.A1 (GND), J1.A12 (GND), J1.B1 (GND), J1.B12 (GND), J1.S1 (SHIELD), J4.6 (VSS), J4.9 (SHIELD), U3.33 (GND), AE1.2 (Shield), C1.2, C10.2, C11.2, C12.2, C13.2, C14.1, C15.2, C2.2, C3.2, C4.2, C5.2, C6.2, C7.2, C8.2, C9.1, J2.4 (Pin_4), J3.13 (GND), J3.8 (GND), R10.1, R2.2, R3.2, R4.2, R9.2, U1.2 (GND), U2.3 (GND), U4.2 (GND), Y1.2, Y1.4
- net RX0: now reaches U3.1 (PB20/RX0/PWM1/CTS1/I2C_SCL)
- net RX0: now also U2.7 (RXD)
- net +3V3: now reaches U3.10 (VDD33)
- net +3V3: now also J4.4 (VDD), U3.11 (VDD33), U3.17 (VDD33), U3.24 (VDD33), U3.31 (VDD33), U3.7 (VDD33), U3.9 (VDD33), C10.1, C11.1, C15.1, C4.1, C6.1, C7.1, C8.1, C9.2, J2.1 (Pin_1), J3.10 (VCC), J3.12 (LED+), R11.1, R12.1, R13.1, R14.1, R15.1, U1.5 (OUT), U2.5 (VCC), U2.8 (V3)
- net at U3.15 (PA4/JTAG_SO/I2C_SDA/PWM4/I2S_BCK/ADC1): now also R1.2, R2.1
- net LCD_RES: now reaches U3.16 (PA7/PWM4/LSPI_MOSI/I2S_MCK/I2S_DI/Touch0)
- net LCD_RES: now also J3.6 (RST)
- net UART3_RX: now reaches U3.18 (PB0/PWM0/LSPI_MISO/TX3/PSRAM_CK/Touch3)
- net UART3_RX: now also J2.3 (Pin_3)
- net UART3_TX: now reaches U3.19 (PB1/PWM1/LSPI_CK/RX3/PSRAM_CS/Touch4)
- net UART3_TX: now also J2.2 (Pin_2)
- net TX0: now reaches U3.2 (PB19/TX0/PWM0/RTS1/I2C_SDA)
- net TX0: now also U2.6 (TXD)
- net LCD_SCK: now reaches U3.20 (PB2/PWM2/LSPI_CK/TX2/PSRAM_D0/Touch5)
- net LCD_SCK: now also J3.4 (SCL)
- net LCD_DC: now reaches U3.21 (PB3/PWM3/LSPI_MISO/RX2/PSRAM_D1/Touch6)
- net LCD_DC: now also J3.5 (DC)
- net LCD_CS: now reaches U3.22 (PB4/LSPI_CS/RTS2/TX4/PSRAM_D2/Touch7)
- net LCD_CS: now also J3.7 (CS)
- net LCD_SDA: now reaches U3.23 (PB5/LSPI_MOSI/CTS2/RX4/PSARM_D3/Touch8)
- net LCD_SDA: now also J3.3 (SDA)
- net at U3.25 (CAP): now also C14.2
- net TF_CLK: now reaches U3.26 (PB6/TX1/MMC_CLK/HSPI_CK/SDIO_CK/Touch9)
- net TF_CLK: now also J4.5 (CLK)
- net TF_CMD: now reaches U3.27 (PB7/RX1/MMC_CMD/HSPI_INT/SDIO_CMD/Touch10)
- net TF_CMD: now also J4.3 (CMD), R11.2
- net TF_DAT0: now reaches U3.28 (PB8/I2S_BCK/MMC_D0/_PWM_BREAK/SDIO_D0/Touch11)
- net TF_DAT0: now also J4.7 (DAT0), R15.2
- net TF_DAT1: now reaches U3.29 (PB9/I2S_LRCK/MMC_D1/_HSPI_CS/SDIO_D1/Touch12)
- net TF_DAT1: now also J4.8 (DAT1), R14.2
- net TF_DAT2: now reaches U3.30 (PB10/I2S_DI/MMC_D2/HSPI_DI/SDIO_D2)
- net TF_DAT2: now also J4.1 (DAT2), R13.2
- net TF_DAT3: now reaches U3.32 (PB11/I2S_DO/MMC_D3/HSPI_DO/SDIO_D3)
- net TF_DAT3: now also J4.2 (DAT3/CD), R12.2
- net RESET: now reaches U3.4 (RESET)
- net RESET: now also C5.1, R5.2
- net at U3.5 (XTAL_OUT): now also C1.1, Y1.3
- net at U3.6 (XTAL_IN): now also C2.1, Y1.1
- net at U3.8 (ANT): now also AE1.1 (A)
- net +5V: now reaches J1.A4 (VBUS), J1.A9 (VBUS), J1.B4 (VBUS), J1.B9 (VBUS)
- net +5V: now also D2.1 (K), R7.2, SW2.1
- net at J1.A5 (CC1): now also R3.1
- net USB_D+: now reaches J1.A6 (D+)
- net USB_D+: now also J1.B6 (D+), U2.1 (UD+)
- net USB_D-: now reaches J1.A7 (D-)
- net USB_D-: now also J1.B7 (D-), U2.2 (UD-)
- net at J1.B5 (CC2): now also R4.1
- new net: C3.1, SW2.2, U1.1 (IN), U1.3 (EN)
- new net: D1.1 (K), U4.1 (CHRG)
- new net: D1.2 (A), R6.1
- new net: R5.1, U2.4 (~{RTS})
- new net: J3.11 (LED-), R10.2
- new net: R6.2, R7.1, R8.2, U4.4 (V+)
- new net: R9.1, U4.5 (PROG)
- new net: C12.1, R8.1
- new net +4V: C13.1, D2.2 (A), R1.1, U4.3 (BAT)
- no-connect marks 0 -> 9
Other:
- note added: "0.96 ISP TFT"
- moved on the sheet: J4, SW1, U3

Commit message: update: 分配封装
Parts:
- removed C15: Cap_0.1uf_0402_16V_X7R, Capacitor_SMD:C_0402_1005Metric, symbol Airm2m_RCL:Cap_0.1uf_0402_16V_X7R
- added C15: 100nf, Capacitor_SMD:C_0402_1005Metric, symbol Device:C
- added D3: SS14, Diode_SMD:D_SMA, symbol Device:D
- added J5: Conn_01x02_Male, Connector_PinHeader_2.54mm:PinHeader_1x02_P2.54mm_Vertical, symbol Connector:Conn_01x02_Male
- D1: footprint (none) -> LED_SMD:LED_0402_1005Metric
- J2: footprint (none) -> Connector_PinHeader_2.54mm:PinHeader_1x04_P2.54mm_Horizontal
- J4: footprint (none) -> chenxuuu_Module:microSD_TF
- R11, R12, R13, R14, R15, R3, R4: footprint (none) -> Resistor_SMD:R_0402_1005Metric
Connections:
- net +3V3: now also C15.1
- net +4V: now also D3.2 (A), J5.1 (Pin_1); no longer D2.2 (A)
- net +5V: now also D2.2 (A); no longer D2.1 (K), SW2.1
- net GND: now also C15.2, J5.2 (Pin_2)
- new net LDO_IN: D2.1 (K), D3.1 (K), SW2.1

Commit message: add: 随便画了画pcb
Parts:
- removed AE1: Antenna_Shield, RF_Antenna:Texas_SWRA117D_2.4GHz_Left, symbol Device:Antenna_Shield
- removed C10, C11, C7: 1uF, Capacitor_SMD:C_0402_1005Metric, symbol Device:C
- removed C6: 104, Capacitor_SMD:C_0402_1005Metric, symbol Device:C
- removed C8: 102, Capacitor_SMD:C_0402_1005Metric, symbol Device:C
- removed C9: 4.7uF, Capacitor_SMD:C_0402_1005Metric, symbol Device:C
- removed J5: Conn_01x02_Male, Connector_PinHeader_2.54mm:PinHeader_1x02_P2.54mm_Vertical, symbol Connector:Conn_01x02_Male
- removed SW2: SW_ON/OFF, symbol Switch:SW_Push
- added SW2: SW_Push_SPDT, chenxuuu_Module:MSK-0002, symbol Switch:SW_Push_SPDT
- added TP1, TP2: TestPoint, TestPoint:TestPoint_Pad_2.0x2.0mm, symbol Connector:TestPoint
- C4: value 10uF -> 1uF
- D2, D3: value SS14 -> MSK4005; footprint Diode_SMD:D_SMA -> Diode_SMD:D_SOD-523
- SW1: value SW_Push -> Side_SWITCH_SW_3*6*3.5mm; footprint (none) -> Button_Switch_SMD:SW_SPST_B3U-3000P-B
Connections:
- net +4V: now also TP1.1
- net GND: now also TP2.1
- net LDO_IN: now also SW2.2 (B)
- net at C3.1, U1.1 (IN), U1.3 (EN): now also SW2.3 (C)
- no-connect marks 9 -> 11
